File: KiCad/ISA8_LPT_COM_RTC.kicad_sch (KiCad schematic)
At the start: 15 parts, among them J1 PRN, J2 Config, U1 82C11, U2 74HCT245, U3 74HCT138, U4 74HCT138

Commit message: Set footprints
Parts:
- removed BUS1: ISA, SKiselev:Conn_Edge_PCB_ISA8, symbol SKiselev:BUSPC_HOST
- added BUS1: BUSPC_DEV, SKiselev:Conn_Edge_PCB_ISA8, symbol SKiselev:BUSPC_DEV
- J2: value Config -> PRN Conf; footprint (none) -> Connector_PinHeader_2.54mm:PinHeader_2x04_P2.54mm_Vertical
- U2: footprint (none) -> Package_DIP:DIP-20_W7.62mm_Socket
- U3, U4: footprint (none) -> Package_DIP:DIP-16_W7.62mm_Socket
Connections:
- net A0: now also BUS1.62 (SA0)
- net A1: now also BUS1.61 (SA1)
- net A2: now also BUS1.60 (SA2)
- net A3: now also BUS1.59 (SA3)
- net A4: now also BUS1.58 (SA4)
- net A5: now also BUS1.57 (SA5)
- net A6: now also BUS1.56 (SA6)
- net A7: now also BUS1.55 (SA7)
- net A8: now also BUS1.54 (SA8)
- net A9: now also BUS1.53 (SA9)
- net AEN: now also BUS1.42 (AEN)
- net D0: now also BUS1.40 (SD0)
- net D1: now also BUS1.39 (SD1)
- net D2: now also BUS1.38 (SD2)
- net D3: now also BUS1.37 (SD3)
- net D4: now also BUS1.36 (SD4)
- net D5: now also BUS1.35 (SD5)
- net D6: now also BUS1.34 (SD6)
- net D7: now also BUS1.33 (SD7)
- net GND: now also BUS1.1 (GND), BUS1.10 (GND), BUS1.31 (GND)
- net IOR: now also BUS1.14 (IOR)
- net IOW: now also BUS1.13 (IOW)
- net IRQ6: now also BUS1.22 (IRQ6)
- net IRQ7: now also BUS1.21 (IRQ7)
- net RESET: now also BUS1.2 (RESET)
- net VCC: now also BUS1.29 (VCC), BUS1.3 (VCC)
- no-connect marks 50 -> 51
Other:
- note added: "Address and IRQ Selection"

Commit message: Design COM ports
Parts:
- removed J2: PRN Conf, Connector_PinHeader_2.54mm:PinHeader_2x04_P2.54mm_Vertical, symbol Connector_Generic:Conn_02x04_Row_Letter_Last
- added BT1: CR2032 cell, SKiselev:Battery_Holder_CR2032_Mouser_122-2420-GR, symbol Device:Battery_Cell
- added C10, C11, C12, C13, C14, C15, C16, C18, C19, C20: 0.1 uF, SKiselev:Cap_Cer_508, symbol Device:C_Small
- added C9: 10 uF, SKiselev:Cap_Elec_Radial_5mm_2.5mm, symbol Device:C_Polarized_Small
- added J2: PRN Conf, Connector_PinHeader_2.54mm:PinHeader_2x04_P2.54mm_Vertical, symbol Connector_Generic:Conn_02x04_Odd_Even
- added J3, J4: Conn_01x10, Connector_PinHeader_2.54mm:PinHeader_2x05_P2.54mm_Vertical, symbol Connector_Generic:Conn_01x10
- added J5: ASYN1 IRQ, Connector_PinHeader_2.54mm:PinHeader_2x02_P2.54mm_Vertical, symbol Connector_Generic:Conn_02x02_Odd_Even
- added J6: ASYN2 IRQ, Connector_PinHeader_2.54mm:PinHeader_2x02_P2.54mm_Vertical, symbol Connector_Generic:Conn_02x02_Odd_Even
- added J7: ASYN1 PORT, Connector_PinHeader_2.54mm:PinHeader_2x02_P2.54mm_Vertical, symbol Connector_Generic:Conn_02x02_Odd_Even
- added J8: ASYN2 PORT, Connector_PinHeader_2.54mm:PinHeader_2x02_P2.54mm_Vertical, symbol Connector_Generic:Conn_02x02_Odd_Even
- added JP1: Clear CMOS, Connector_PinHeader_2.54mm:PinHeader_1x02_P2.54mm_Vertical, symbol Jumper:Jumper_2_Open
- added P1: DE9, SKiselev:Conn_Dsub_DE9M, symbol SKiselev:DE9
- added QG1: OSC, symbol SKiselev:OSC
- added RN1: 10k, SKiselev:Conn_SIL5, symbol Device:R_Network04
- added SW1: Switch_DIP_3_Positions, SKiselev:Switch_DIP_3_Positions, symbol SKiselev:Switch_DIP_3_Positions
- added U10, U8: GD75232N, Package_DIP:DIP-20_W7.62mm, symbol Interface_UART:GD75232N
- added U5: DS12885, Package_DIP:DIP-24_W15.24mm_Socket, symbol SKiselev:DS12885
- added U6: ATF16V8B, Package_DIP:DIP-20_W7.62mm_Socket, symbol SKiselev:ATF16V8B
- added U7, U9: 16550, Package_LCC:PLCC-44_THT-Socket, symbol SKiselev:16550-PLCC
- added Y1: 32768Hz, SKiselev:Crystal_32K_Horiz, symbol Device:Crystal_GND3
- C1, C2, C3, C4, C5, C6, C7, C8: footprint Capacitor_THT:C_Disc_D5.1mm_W3.2mm_P5.00mm -> Capacitor_THT:C_Disc_D5.0mm_W2.5mm_P5.00mm
- U3: renamed from U1; footprint Package_DIP:DIP-40_W25.4mm_Socket -> Package_DIP:DIP-40_W15.24mm_Socket
- renumbered U3 to U1, U4 to U2, U2 to U4
Connections:
- net 0x278: now also J2.5 (Pin_5)
- net 0x2E8: now also J8.3 (Pin_3)
- net 0x2F8: now also J7.3 (Pin_3)
- net 0x378: now also J2.7 (Pin_7)
- net 0x3E8: now also J8.1 (Pin_1)
- net 0x3F8: now also J7.1 (Pin_1)
- net A0: now also U6.1 (I/CLK), U7.31 (A0), U9.31 (A0)
- net A1: now also U7.30 (A1), U9.30 (A1)
- net A2: now also U6.2 (I1), U7.29 (A2), U9.29 (A2)
- net A3: now also U6.3 (I2)
- net A4: now also U6.4 (I3)
- net A5: now also U6.5 (I4)
- net A6: now also U6.6 (I5)
- net A7: now also U6.7 (I6)
- net A8: now also U6.8 (I7)
- net A9: now also U6.9 (I8)
- net AEN: now also U6.17 (I/O3)
- net D0: now also U5.4 (AD0), U7.2 (D0), U9.2 (D0)
- net D1: now also U5.5 (AD1), U7.3 (D1), U9.3 (D1)
- net D2: now also U5.6 (AD2), U7.4 (D2), U9.4 (D2)
- net D3: now also U5.7 (AD3), U7.5 (D3), U9.5 (D3)
- net D4: now also U5.8 (AD4), U7.6 (D4), U9.6 (D4)
- net D5: now also U5.9 (AD5), U7.7 (D5), U9.7 (D5)
- net D6: now also U5.10 (AD6), U7.8 (D6), U9.8 (D6)
- net D7: now also U5.11 (AD7), U7.9 (D7), U9.9 (D7)
- net GND: now also BT1.2 (-), C10.2, C11.2, C12.2, C13.2, C14.2, C15.2, C16.2, C18.2, C19.2, C20.2, C9.2, J3.5 (Pin_5), J4.5 (Pin_5), JP1.2 (B), P1.5, QG1.7 (GND), SW1.1, SW1.2, SW1.3, U10.11 (GND), U5.12 (GND), U5.13 (~{CS}), U5.16 (GND), U6.10 (GND), U7.21 (WR), U7.22 (GND), U7.25 (RD), U7.28 (~{ADS}), U8.11 (GND), U9.21 (WR), U9.22 (GND), U9.25 (RD), U9.28 (~{ADS}), Y1.3
- net IOR: now also U6.13 (I/O7), U7.24 (~{RD}), U9.24 (~{RD})
- net IOW: now also U6.12 (I/O8), U7.20 (~{WR}), U9.20 (~{WR})
- net IRQ6: now also J2.1 (Pin_1)
- net IRQ7: now also J2.3 (Pin_3)
- net PRN_CS: now also J2.6 (Pin_6), J2.8 (Pin_8)
- net PRN_IRQ: now also J2.2 (Pin_2), J2.4 (Pin_4)
- net RESET: now also U7.39 (MR), U9.39 (MR)
- net VCC: now also C10.1, C11.1, C12.1, C13.1, C14.1, C15.1, C16.1, C18.1, C19.1, C20.1, C9.1, QG1.14 (VCC), RN1.1 (common), U10.20 (V_{CC}), U5.18 (~{RESET}), U5.24 (VCC), U6.20 (VCC), U7.14 (CS0), U7.15 (CS1), U7.44 (VCC), U8.20 (V_{CC}), U9.14 (CS0), U9.15 (CS1), U9.44 (VCC)
- net VSS: now reaches BUS1.7 (-12V)
- net VSS: now also U10.10 (V_{SS}), U8.10 (V_{SS})
- net VDD: now reaches BUS1.9 (+12V)
- net VDD: now also U10.1 (V_{DD}), U8.1 (V_{DD})
- new net: U9.10 (RCLK), U9.17 (~{BAUDOUT})
- new net: U10.17 (RY3), U9.11 (SIN)
- new net: U10.15 (DA2), U9.13 (SOUT)
- new net: QG1.8 (OUT), U7.18 (XIN), U9.18 (XIN)
- new net: U10.16 (DA1), U9.36 (~{RTS})
- new net: U10.13 (DA3), U9.37 (~{DTR})
- new net: U10.14 (RY4), U9.40 (~{CTS})
- new net: U10.18 (RY2), U9.41 (~{DSR})
- new net: U10.19 (RY1), U9.42 (~{DCD})
- new net: U10.12 (RY5), U9.43 (~{RI})
- new net: JP1.1 (A), U5.21 (~{RCLR})
- new net: BT1.1 (+), U5.20 (VBAT)
- new net: U5.2 (X1), Y1.1
- new net: U5.3 (X2), Y1.2
- new net: J4.1 (Pin_1), U10.2 (RA1)
- new net: J4.2 (Pin_2), U10.4 (RA3)
- new net: J4.3 (Pin_3), U10.6 (DY2)
- new net: J4.4 (Pin_4), U10.8 (DY3)
- new net: J4.6 (Pin_6), U10.3 (RA2)
- new net: J4.7 (Pin_7), U10.5 (DY1)
- new net: J4.8 (Pin_8), U10.7 (RA4)
- new net: J4.9 (Pin_9), U10.9 (RA5)
- new net: U7.43 (~{RI}), U8.12 (RY5)
- new net: U7.37 (~{DTR}), U8.13 (DA3)
- new net: U7.40 (~{CTS}), U8.14 (RY4)
- new net: U7.13 (SOUT), U8.15 (DA2)
- new net: U7.36 (~{RTS}), U8.16 (DA1)
- new net: U7.11 (SIN), U8.17 (RY3)
- new net: U7.41 (~{DSR}), U8.18 (RY2)
- new net: U7.42 (~{DCD}), U8.19 (RY1)
- new net: J3.1 (Pin_1), P1.1, U8.2 (RA1)
- new net: J3.6 (Pin_6), P1.6 (P6), U8.3 (RA2)
- new net: J3.2 (Pin_2), P1.2, U8.4 (RA3)
- new net: J3.7 (Pin_7), P1.7 (P7), U8.5 (DY1)
- new net: J3.3 (Pin_3), P1.3, U8.6 (DY2)
- new net: J3.8 (Pin_8), P1.8 (P8), U8.7 (RA4)
- new net: J3.4 (Pin_4), P1.4, U8.8 (DY3)
- new net: J3.9 (Pin_9), P1.9 (P9), U8.9 (RA5)
- new net: U7.10 (RCLK), U7.17 (~{BAUDOUT})
- new net AS0: RN1.2 (R1), SW1.6, U6.19 (I/O1)
- new net AS1: RN1.3 (R2), SW1.5, U6.18 (I/O2)
- new net AS2: RN1.4 (R3), SW1.4, U6.11 (I9/~{OE})
- new net IRQ3: J5.1 (Pin_1), J6.1 (Pin_1)
- new net IRQ4: J5.3 (Pin_3), J6.3 (Pin_3)
- new net RTCALE: U5.14 (AS), U6.14 (I/O6)
- new net RTCRD: U5.17 (DS), U6.16 (I/O4)
- new net RTCWR: U5.15 (R/~{W}), U6.15 (I/O5)
- new net UART_CS1: J7.2 (Pin_2), J7.4 (Pin_4), U7.16 (~{CS2})
- new net UART_CS2: J8.2 (Pin_2), J8.4 (Pin_4), U9.16 (~{CS2})
- new net UART_IRQ1: J5.2 (Pin_2), J5.4 (Pin_4), U7.33 (INTR)
- new net UART_IRQ2: J6.2 (Pin_2), J6.4 (Pin_4), U9.33 (INTR)
- new net ~{RTC_IRQ}: RN1.5 (R4), U5.19 (~{IRQ})
- no-connect marks 51 -> 62
Other:
- note added: "Capacitors"
- note added: "Real Time Clock"
- title: LPT Isa Card -> ISA PC Card with 1 LPT and 2 COM ports and RTC
- moved on the sheet: BUS1, C1, C2, C3, C4, C5, C6, C7, C8, J1, U1, U2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
